File: STM32_NRF24.sch (KiCad schematic (older format))
At the start: 1 part

Commit message: upd
Parts:
- added C? (x2): 1u, Capacitors_SMD:C_0805, symbol C_Cer_SMD_0805
- added C? (x3): 100n, Capacitors_SMD:C_0805, symbol C_Cer_SMD_0805
- added D?: PWR_LED, symbol Led_Small
- added P?: CONN_BOOT, symbol CONN_01X02
- added P?: CONN_SWD, symbol CONN_01X04
- added R? (x3): 1K, Resistors_SMD:R_0805, symbol R_SMD_0805
- added SW?: SW_RST, symbol SW_PUSH
- added U?: nRF24L01_MODULE, BK_Common:NRF24L01_MODULE, symbol nRF24L01_MODULE
Connections:
- net labels added: +3.3V, 485_DE, BOOT0, DE, GND, NRST, PW_CF, PW_CF1, PW_SEL, RF_CE, RF_IRQ, RF_POW, RX, SPI1_MISO, SPI1_MOSI, SPI1_NSS, SPI1_SCK, SYS_SWCLK, SYS_SWDIO, TX, USART_RX, USART_TX
- wire segments 0 -> 62
- no-connect marks 0 -> 1
Other:
- moved on the sheet: U?
