File: HW/PWRMET_24G.sch (KiCad schematic (older format))
At the start: 0 parts

Commit message: PCB Start
Connections:
- no-connect marks 1 -> 0
Changed lines of the file:
@@
 LIBS:stm32
 LIBS:BK_Common
-LIBS:BK_LED_Drivers
-LIBS:BK_STM8
 LIBS:PWRMET_24G-cache
 EELAYER 25 0
@@
 Wire Wire Line
 	3450 4325 3050 4325
-Wire Wire Line
-	2125 2425 2000 2425
-NoConn ~ 2000 2425
 $EndSCHEMATC
