File: HW/RS485_ISOL.sch (KiCad schematic (older format))
At the start: 19 parts

Commit message: PCB Start
Parts:
- P5: renamed from P?; footprint (none) -> Pin_Headers:Pin_Header_Straight_1x04_Pitch2.54mm
- U4, U6, U8: renamed from U?; footprint DIP-4 -> Housings_DIP:DIP-4_W9.53mm_SMD
- U7: renamed from U?; footprint SOT-89 -> TO_SOT_Packages_SMD:SOT-89-3
- gave numbers to parts that had none: 14
Other:
- moved on the sheet: C10, C11, C12, C9, R20, R21, R22, R23, R24, R25, R26, R27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

Commit message: PCB Upd
Other:
- moved on the sheet: R20, R24
Changed lines of the file:
@@
 DI
 Wire Wire Line
-	7075 1800 7475 1800
-Wire Wire Line
 	7075 1900 7825 1900
 Wire Wire Line
 	7075 2000 7825 2000
-Wire Wire Line
-	7075 2100 7475 2100
-Text Label 7275 1800 0    60   ~ 0
+Text Label 7100 1800 0    60   ~ 0
 PISO
 Text Label 7775 1900 0    60   ~ 0
@@
 Text Label 7775 2000 0    60   ~ 0
 A
-Text Label 7275 2100 0    60   ~ 0
+Text Label 7100 2100 0    60   ~ 0
 GISO
 Wire Wire Line
@@
 L R_SMD_0805 R20
 U 1 1 5921EE6D
-P 7275 1500
-F 0 "R20" V 7350 1450 50  0000 L CNN
-F 1 "20K" V 7200 1425 50  0000 L CNN
-F 2 "Resistors_SMD:R_0805" H 7325 1350 50  0001 C CNN
-F 3 "" H 7275 1500 50  0000 C CNN
-	1    7275 1500
+P 7475 1500
+F 0 "R20" V 7550 1450 50  0000 L CNN
+F 1 "20K" V 7400 1425 50  0000 L CNN
+F 2 "Resistors_SMD:R_0805" H 7525 1350 50  0001 C CNN
+F 3 "" H 7475 1500 50  0000 C CNN
+	1    7475 1500
 	-1   0    0    1
 $EndComp
 Wire Wire Line
-	7275 1400 7275 1300
-Wire Wire Line
-	7275 1300 7475 1300
-Wire Wire Line
-	7275 1600 7275 2000
-Connection ~ 7275 2000
-Text Label 7275 1300 0    60   ~ 0
+	7475 1400 7475 1300
+Wire Wire Line
+	7475 1300 7675 1300
+Text Label 7475 1300 0    60   ~ 0
 PISO
 $Comp
 L R_SMD_0805 R24
 U 1 1 5921EF8C
-P 7225 2400
-F 0 "R24" V 7300 2350 50  0000 L CNN
-F 1 "20K" V 7150 2325 50  0000 L CNN
-F 2 "Resistors_SMD:R_0805" H 7275 2250 50  0001 C CNN
-F 3 "" H 7225 2400 50  0000 C CNN
-	1    7225 2400
+P 7375 2400
+F 0 "R24" V 7450 2350 50  0000 L CNN
+F 1 "20K" V 7300 2325 50  0000 L CNN
+F 2 "Resistors_SMD:R_0805" H 7425 2250 50  0001 C CNN
+F 3 "" H 7375 2400 50  0000 C CNN
+	1    7375 2400
 	-1   0    0    1
 $EndComp
 Wire Wire Line
-	7225 2300 7225 1900
-Connection ~ 7225 1900
-Wire Wire Line
-	7225 2500 7225 2650
-Wire Wire Line
-	7225 2650 7475 2650
-Text Label 7275 2650 0    60   ~ 0
+	7375 2500 7375 2650
+Wire Wire Line
+	7375 2650 7625 2650
+Text Label 7425 2650 0    60   ~ 0
 GISO
 $Comp
@@
 	6175 2000 6175 1900
 Connection ~ 6175 1900
+Wire Wire Line
+	7075 1800 7300 1800
+Wire Wire Line
+	7075 2100 7300 2100
+Wire Wire Line
+	7375 2300 7375 1900
+Connection ~ 7375 1900
+Wire Wire Line
+	7475 1600 7475 2000
+Connection ~ 7475 2000
 $EndSCHEMATC
