File: HW/STM32_NRF24.sch (KiCad schematic (older format))
At the start: 14 parts

Commit message: PCB Start
Parts:
- D1: renamed from D?; footprint (none) -> LEDs:LED_0805
- P1: renamed from P?; footprint (none) -> Pin_Headers:Pin_Header_Straight_1x02_Pitch2.54mm
- P2: renamed from P?; footprint (none) -> Pin_Headers:Pin_Header_Straight_1x04_Pitch2.54mm
- SW1: renamed from SW?; footprint (none) -> BK_Common:SW_SPST_TACT_SMD_3X6
- gave numbers to parts that had none: 10
Changed lines of the file:
@@
 LIBS:stm32
 LIBS:BK_Common
-LIBS:BK_LED_Drivers
-LIBS:BK_STM8
 LIBS:PWRMET_24G-cache
 EELAYER 25 0
@@
 $EndDescr
 $Comp
-L STM32F030F4Px U?
+L STM32F030F4Px U1
 U 1 1 591CC106
 P 6475 2575
-F 0 "U?" H 4875 3500 50  0000 L BNN
+F 0 "U1" H 4875 3500 50  0000 L BNN
 F 1 "STM32F030F4Px" H 8075 3500 50  0000 R BNN
 F 2 "Housings_SSOP:TSSOP-20_4.4x6.5mm_Pitch0.65mm" H 8075 3450 50  0001 R TNN
@@
 BOOT0
 $Comp
-L C_Cer_SMD_0805 C?
+L C_Cer_SMD_0805 C1
 U 1 1 5920FE5F
 P 6675 1275
-F 0 "C?" H 6685 1345 50  0000 L CNN
+F 0 "C1" H 6685 1345 50  0000 L CNN
 F 1 "1u" H 6685 1195 50  0000 L CNN
 F 2 "Capacitors_SMD:C_0805" H 6675 1125 50  0001 C CNN
@@
 $EndComp
 $Comp
-L C_Cer_SMD_0805 C?
+L C_Cer_SMD_0805 C2
 U 1 1 5920FEBD
 P 6875 1275
-F 0 "C?" H 6885 1345 50  0000 L CNN
+F 0 "C2" H 6885 1345 50  0000 L CNN
 F 1 "100n" H 6885 1195 50  0000 L CNN
 F 2 "Capacitors_SMD:C_0805" H 6875 1125 50  0001 C CNN
@@
 $EndComp
 $Comp
-L GND #PWR?
+L GND #PWR01
 U 1 1 5920FF27
 P 6775 1500
-F 0 "#PWR?" H 6775 1250 50  0001 C CNN
+F 0 "#PWR01" H 6775 1250 50  0001 C CNN
 F 1 "GND" H 6775 1350 50  0000 C CNN
 F 2 "" H 6775 1500 50  0000 C CNN
@@
 $EndComp
 $Comp
-L +3.3V #PWR?
+L +3.3V #PWR02
 U 1 1 5920FF6B
 P 6375 1025
-F 0 "#PWR?" H 6375 875 50  0001 C CNN
+F 0 "#PWR02" H 6375 875 50  0001 C CNN
 F 1 "+3.3V" H 6375 1165 50  0000 C CNN
 F 2 "" H 6375 1025 50  0000 C CNN
@@
 $EndComp
 $Comp
-L R_SMD_0805 R?
+L R_SMD_0805 R2
 U 1 1 5921003E
 P 2400 2450
-F 0 "R?" H 2430 2470 50  0000 L CNN
+F 0 "R2" H 2430 2470 50  0000 L CNN
 F 1 "1K" H 2430 2410 50  0000 L CNN
 F 2 "Resistors_SMD:R_0805" H 2450 2300 50  0001 C CNN
@@
 $EndComp
 $Comp
-L C_Cer_SMD_0805 C?
+L C_Cer_SMD_0805 C3
 U 1 1 592100AD
 P 2400 3050
-F 0 "C?" H 2410 3120 50  0000 L CNN
+F 0 "C3" H 2410 3120 50  0000 L CNN
 F 1 "100n" H 2410 2970 50  0000 L CNN
 F 2 "Capacitors_SMD:C_0805" H 2400 2900 50  0001 C CNN
@@
 $EndComp
 $Comp
-L SW_PUSH SW?
+L SW_PUSH SW1
 U 1 1 5921013F
 P 2050 3050
-F 0 "SW?" H 2200 3160 50  0000 C CNN
+F 0 "SW1" H 2200 3160 50  0000 C CNN
 F 1 "SW_RST" H 2050 2970 50  0000 C CNN
-F 2 "" H 2050 3050 50  0000 C CNN
+F 2 "BK_Common:SW_SPST_TACT_SMD_3X6" H 2050 3050 50  0001 C CNN
 F 3 "" H 2050 3050 50  0000 C CNN
 	1    2050 3050
@@
 $EndComp
 $Comp
-L +3.3V #PWR?
+L +3.3V #PWR03
 U 1 1 59210451
 P 2400 2250
-F 0 "#PWR?" H 2400 2100 50  0001 C CNN
+F 0 "#PWR03" H 2400 2100 50  0001 C CNN
 F 1 "+3.3V" H 2400 2390 50  0000 C CNN
 F 2 "" H 2400 2250 50  0000 C CNN
@@
 $EndComp
 $Comp
-L GND #PWR?
+L GND #PWR04
 U 1 1 592104BE
 P 2400 3550
-F 0 "#PWR?" H 2400 3300 50  0001 C CNN
+F 0 "#PWR04" H 2400 3300 50  0001 C CNN
 F 1 "GND" H 2400 3400 50  0000 C CNN
 F 2 "" H 2400 3550 50  0000 C CNN
@@
 $EndComp
 $Comp
-L Led_Small D?
+L Led_Small D1
 U 1 1 59210531
 P 2900 3050
-F 0 "D?" H 2850 3175 50  0000 L CNN
+F 0 "D1" H 2850 3175 50  0000 L CNN
 F 1 "PWR_LED" H 2725 2950 50  0000 L CNN
-F 2 "" V 2900 3050 50  0000 C CNN
+F 2 "LEDs:LED_0805" V 2900 3050 50  0001 C CNN
 F 3 "" V 2900 3050 50  0000 C CNN
 	1    2900 3050
@@
 $EndComp
 $Comp
-L R_SMD_0805 R?
+L R_SMD_0805 R3
 U 1 1 5921058B
 P 2900 2450
-F 0 "R?" H 2930 2470 50  0000 L CNN
+F 0 "R3" H 2930 2470 50  0000 L CNN
 F 1 "1K" H 2930 2410 50  0000 L CNN
 F 2 "Resistors_SMD:R_0805" H 2950 2300 50  0001 C CNN
@@
 $EndComp
 $Comp
-L +3.3V #PWR?
+L +3.3V #PWR05
 U 1 1 592105BF
 P 2900 2250
-F 0 "#PWR?" H 2900 2100 50  0001 C CNN
+F 0 "#PWR05" H 2900 2100 50  0001 C CNN
 F 1 "+3.3V" H 2900 2390 50  0000 C CNN
 F 2 "" H 2900 2250 50  0000 C CNN
@@
 $EndComp
 $Comp
-L GND #PWR?
+L GND #PWR06
 U 1 1 592105E2
 P 2900 3550
-F 0 "#PWR?" H 2900 3300 50  0001 C CNN
+F 0 "#PWR06" H 2900 3300 50  0001 C CNN
 F 1 "GND" H 2900 3400 50  0000 C CNN
 F 2 "" H 2900 3550 50  0000 C CNN
@@
 NRST
 $Comp
-L CONN_01X02 P?
+L CONN_01X02 P1
 U 1 1 59210766
 P 1150 3050
-F 0 "P?" H 1150 3200 50  0000 C CNN
+F 0 "P1" H 1150 3200 50  0000 C CNN
 F 1 "CONN_BOOT" V 1250 3050 50  0000 C CNN
-F 2 "" H 1150 3050 50  0000 C CNN
+F 2 "Pin_Headers:Pin_Header_Straight_1x02_Pitch2.54mm" H 1150 3050 50  0001 C CNN
 F 3 "" H 1150 3050 50  0000 C CNN
 	1    1150 3050
@@
 $EndComp
 $Comp
-L R_SMD_0805 R?
+L R_SMD_0805 R1
 U 1 1 592107CC
 P 1350 2450
-F 0 "R?" H 1380 2470 50  0000 L CNN
+F 0 "R1" H 1380 2470 50  0000 L CNN
 F 1 "1K" H 1380 2410 50  0000 L CNN
 F 2 "Resistors_SMD:R_0805" H 1400 2300 50  0001 C CNN
@@
 $EndComp
 $Comp
-L +3.3V #PWR?
+L +3.3V #PWR07
 U 1 1 59210816
 P 1350 2250
-F 0 "#PWR?" H 1350 2100 50  0001 C CNN
+F 0 "#PWR07" H 1350 2100 50  0001 C CNN
 F 1 "+3.3V" H 1350 2390 50  0000 C CNN
 F 2 "" H 1350 2250 50  0000 C CNN
@@
 $EndComp
 $Comp
-L GND #PWR?
+L GND #PWR08
 U 1 1 5921083F
 P 1350 3550
-F 0 "#PWR?" H 1350 3300 50  0001 C CNN
+F 0 "#PWR08" H 1350 3300 50  0001 C CNN
 F 1 "GND" H 1350 3400 50  0000 C CNN
 F 2 "" H 1350 3550 50  0000 C CNN
@@
 RF_CE
 $Comp
-L GND #PWR?
+L GND #PWR09
 U 1 1 5921142D
 P 6475 3575
-F 0 "#PWR?" H 6475 3325 50  0001 C CNN
+F 0 "#PWR09" H 6475 3325 50  0001 C CNN
 F 1 "GND" H 6475 3425 50  0000 C CNN
 F 2 "" H 6475 3575 50  0000 C CNN
@@
 SPI1_NSS
 $Comp
-L nRF24L01_MODULE U?
+L nRF24L01_MODULE U2
 U 1 1 5921521D
 P 6450 4950
-F 0 "U?" H 6700 5400 60  0000 C CNN
+F 0 "U2" H 6700 5400 60  0000 C CNN
 F 1 "nRF24L01_MODULE" H 6900 4500 60  0000 C CNN
 F 2 "BK_Common:NRF24L01_MODULE" H 6450 4300 60  0001 C CNN
@@
 $EndComp
 $Comp
-L GND #PWR?
+L GND #PWR010
 U 1 1 59215406
 P 6450 5700
-F 0 "#PWR?" H 6450 5450 50  0001 C CNN
+F 0 "#PWR010" H 6450 5450 50  0001 C CNN
 F 1 "GND" H 6450 5550 50  0000 C CNN
 F 2 "" H 6450 5700 50  0000 C CNN
@@
 $EndComp
 $Comp
-L C_Cer_SMD_0805 C?
+L C_Cer_SMD_0805 C4
 U 1 1 5921565F
 P 7025 4225
-F 0 "C?" H 7035 4295 50  0000 L CNN
+F 0 "C4" H 7035 4295 50  0000 L CNN
 F 1 "1u" H 7035 4145 50  0000 L CNN
 F 2 "Capacitors_SMD:C_0805" H 7025 4075 50  0001 C CNN
@@
 $EndComp
 $Comp
-L C_Cer_SMD_0805 C?
+L C_Cer_SMD_0805 C5
 U 1 1 592156F3
 P 7225 4225
-F 0 "C?" H 7235 4295 50  0000 L CNN
+F 0 "C5" H 7235 4295 50  0000 L CNN
 F 1 "100n" H 7235 4145 50  0000 L CNN
 F 2 "Capacitors_SMD:C_0805" H 7225 4075 50  0001 C CNN
@@
 $EndComp
 $Comp
-L GND #PWR?
+L GND #PWR011
 U 1 1 59215774
 P 7125 4500
-F 0 "#PWR?" H 7125 4250 50  0001 C CNN
+F 0 "#PWR011" H 7125 4250 50  0001 C CNN
 F 1 "GND" H 7125 4350 50  0000 C CNN
 F 2 "" H 7125 4500 50  0000 C CNN
@@
 $EndComp
 $Comp
-L +3.3V #PWR?
+L +3.3V #PWR012
 U 1 1 592157B3
 P 7125 3975
-F 0 "#PWR?" H 7125 3825 50  0001 C CNN
+F 0 "#PWR012" H 7125 3825 50  0001 C CNN
 F 1 "+3.3V" H 7125 4115 50  0000 C CNN
 F 2 "" H 7125 3975 50  0000 C CNN
@@
 SPI1_NSS
 $Comp
-L CONN_01X04 P?
+L CONN_01X04 P2
 U 1 1 592162DE
 P 10600 4300
-F 0 "P?" H 10600 4550 50  0000 C CNN
+F 0 "P2" H 10600 4550 50  0000 C CNN
 F 1 "CONN_SWD" V 10700 4300 50  0000 C CNN
-F 2 "" H 10600 4300 50  0000 C CNN
+F 2 "Pin_Headers:Pin_Header_Straight_1x04_Pitch2.54mm" H 10600 4300 50  0001 C CNN
 F 3 "" H 10600 4300 50  0000 C CNN
 	1    10600 4300
@@
 $EndComp
 $Comp
-L +3.3V #PWR?
+L +3.3V #PWR013
 U 1 1 592163B5
 P 10225 3975
-F 0 "#PWR?" H 10225 3825 50  0001 C CNN
+F 0 "#PWR013" H 10225 3825 50  0001 C CNN
 F 1 "+3.3V" H 10225 4115 50  0000 C CNN
 F 2 "" H 10225 3975 50  0000 C CNN
@@
 $EndComp
 $Comp
-L GND #PWR?
+L GND #PWR014
 U 1 1 592163EA
 P 10250 4675
-F 0 "#PWR?" H 10250 4425 50  0001 C CNN
+F 0 "#PWR014" H 10250 4425 50  0001 C CNN
 F 1 "GND" H 10250 4525 50  0000 C CNN
 F 2 "" H 10250 4675 50  0000 C CNN

Commit message: SCH&PCB Update
Parts:
- added D2: PLS_LED, LEDs:LED_D5.0mm, symbol Led_Small
- added R29: 1K, Resistors_SMD:R_0805, symbol R_SMD_0805
Connections:
- net labels added: PLS_OUT
- net labels removed: RF_POW
- wire segments 62 -> 66
- no-connect marks 1 -> 0
Changed lines of the file:
@@
 LIBS:stm32
 LIBS:BK_Common
+LIBS:BK_LED_Drivers
+LIBS:BK_STM8
 LIBS:PWRMET_24G-cache
 EELAYER 25 0
@@
 Text Label 8325 2275 0    60   ~ 0
 USART_RX
-Text Label 4375 2875 0    60   ~ 0
-RF_POW
 Text Label 4375 2775 0    60   ~ 0
 485_DE
@@
 Text Label 9975 4350 0    60   ~ 0
 SYS_SWCLK
-NoConn ~ 4375 2875
 Text HLabel 8825 2775 2    60   Input ~ 0
 PW_CF
@@
 Connection ~ 6875 1475
 Connection ~ 6875 1100
+Text Label 4375 2875 0    60   ~ 0
+PLS_OUT
+$Comp
+L R_SMD_0805 R29
+U 1 1 592A4032
+P 3200 2450
+F 0 "R29" H 3230 2470 50  0000 L CNN
+F 1 "1K" H 3230 2410 50  0000 L CNN
+F 2 "Resistors_SMD:R_0805" H 3250 2300 50  0001 C CNN
+F 3 "" H 3200 2450 50  0000 C CNN
+	1    3200 2450
+	1    0    0    -1
+$EndComp
+$Comp
+L Led_Small D2
+U 1 1 592A4087
+P 3200 3025
+F 0 "D2" H 3150 3150 50  0000 L CNN
+F 1 "PLS_LED" H 3025 2925 50  0000 L CNN
+F 2 "LEDs:LED_D5.0mm" V 3200 3025 50  0001 C CNN
+F 3 "" V 3200 3025 50  0000 C CNN
+	1    3200 3025
+	0    -1   -1   0
+$EndComp
+$Comp
+L GND #PWR015
+U 1 1 592A40D3
+P 3200 3550
+F 0 "#PWR015" H 3200 3300 50  0001 C CNN
+F 1 "GND" H 3200 3400 50  0000 C CNN
+F 2 "" H 3200 3550 50  0000 C CNN
+F 3 "" H 3200 3550 50  0000 C CNN
+	1    3200 3550
+	1    0    0    -1
+$EndComp
+Wire Wire Line
+	3200 3125 3200 3550
+Wire Wire Line
+	3200 2925 3200 2550
+Wire Wire Line
+	3200 2350 3200 2200
+Wire Wire Line
+	3200 2200 3550 2200
+Text Label 3200 2200 0    60   ~ 0
+PLS_OUT
 $EndSCHEMATC
