File: HW/HLW8012.sch (KiCad schematic (older format))
At the start: 23 parts

Commit message: PCB Start
Parts:
- added R6: 0.001R, Resistors_SMD:R_2512_HandSoldering, symbol R_SMD_1206
- P3, P4: renamed from P?; footprint (none) -> Terminal_Blocks:TerminalBlock_Pheonix_MKDS1.5-2pol
- PS1: renamed from PS?; footprint 5V 700mA PS -> BK_Common:SWPSU_5V_700mA
- Q1: renamed from Q?; footprint (none) -> TO_SOT_Packages_SMD:SOT-23
- R7: renamed from R?; footprint Resistors_SMD:R_1206 -> BK_Common:Shunt_l10mm_d2mm
- gave numbers to parts that had none: 18
Connections:
- wire segments 55 -> 57

Commit message: SCH&PCB Update
Changed lines of the file:
@@
 LIBS:stm32
 LIBS:BK_Common
+LIBS:BK_LED_Drivers
+LIBS:BK_STM8
 LIBS:PWRMET_24G-cache
 EELAYER 25 0
@@
 Connection ~ 1500 3200
 $Comp
-L GND #PWR015
+L GND #PWR016
 U 1 1 591C1799
 P 1500 3325
-F 0 "#PWR015" H 1500 3075 50  0001 C CNN
+F 0 "#PWR016" H 1500 3075 50  0001 C CNN
 F 1 "GND" H 1500 3175 50  0000 C CNN
 F 2 "" H 1500 3325 50  0000 C CNN
@@
 	4350 2025 4350 1675
 $Comp
-L GND #PWR016
+L GND #PWR017
 U 1 1 591C286E
 P 4150 1875
-F 0 "#PWR016" H 4150 1625 50  0001 C CNN
+F 0 "#PWR017" H 4150 1625 50  0001 C CNN
 F 1 "GND" H 4150 1725 50  0000 C CNN
 F 2 "" H 4150 1875 50  0000 C CNN
@@
 V1N
 $Comp
-L GND #PWR017
+L GND #PWR018
 U 1 1 591C529B
 P 3725 2475
-F 0 "#PWR017" H 3725 2225 50  0001 C CNN
+F 0 "#PWR018" H 3725 2225 50  0001 C CNN
 F 1 "GND" H 3725 2325 50  0000 C CNN
 F 2 "" H 3725 2475 50  0000 C CNN
@@
 LD_Back
 $Comp
-L +5V #PWR018
+L +5V #PWR019
 U 1 1 591C689E
 P 7125 4350
-F 0 "#PWR018" H 7125 4200 50  0001 C CNN
+F 0 "#PWR019" H 7125 4200 50  0001 C CNN
 F 1 "+5V" H 7125 4490 50  0000 C CNN
 F 2 "" H 7125 4350 50  0000 C CNN
@@
 	7125 4350 7125 4400
 $Comp
-L GND #PWR019
+L GND #PWR020
 U 1 1 591C6A3D
 P 7125 5600
-F 0 "#PWR019" H 7125 5350 50  0001 C CNN
+F 0 "#PWR020" H 7125 5350 50  0001 C CNN
 F 1 "GND" H 7125 5450 50  0000 C CNN
 F 2 "" H 7125 5600 50  0000 C CNN
@@
 	8550 5475 8550 5600
 $Comp
-L GND #PWR020
+L GND #PWR021
 U 1 1 591C6EC8
 P 8275 5600
-F 0 "#PWR020" H 8275 5350 50  0001 C CNN
+F 0 "#PWR021" H 8275 5350 50  0001 C CNN
 F 1 "GND" H 8275 5450 50  0000 C CNN
 F 2 "" H 8275 5600 50  0000 C CNN
@@
 $EndComp
 $Comp
-L GND #PWR021
+L GND #PWR022
 U 1 1 591C6F0C
 P 8550 5600
-F 0 "#PWR021" H 8550 5350 50  0001 C CNN
+F 0 "#PWR022" H 8550 5350 50  0001 C CNN
 F 1 "GND" H 8550 5450 50  0000 C CNN
 F 2 "" H 8550 5600 50  0000 C CNN
@@
 $EndComp
 $Comp
-L +5V #PWR022
+L +5V #PWR023
 U 1 1 591D3A25
 P 9175 4350
-F 0 "#PWR022" H 9175 4200 50  0001 C CNN
+F 0 "#PWR023" H 9175 4200 50  0001 C CNN
 F 1 "+5V" H 9175 4490 50  0000 C CNN
 F 2 "" H 9175 4350 50  0000 C CNN
@@
 $EndComp
 $Comp
-L GND #PWR023
+L GND #PWR024
 U 1 1 591D3D63
 P 9175 5600
-F 0 "#PWR023" H 9175 5350 50  0001 C CNN
+F 0 "#PWR024" H 9175 5350 50  0001 C CNN
 F 1 "GND" H 9175 5450 50  0000 C CNN
 F 2 "" H 9175 5600 50  0000 C CNN
@@
 	8650 2700 8650 2875
 $Comp
-L GND #PWR024
+L GND #PWR025
 U 1 1 591D5193
 P 8650 2875
-F 0 "#PWR024" H 8650 2625 50  0001 C CNN
+F 0 "#PWR025" H 8650 2625 50  0001 C CNN
 F 1 "GND" H 8650 2725 50  0000 C CNN
 F 2 "" H 8650 2875 50  0000 C CNN
@@
 $EndComp
 $Comp
-L +5V #PWR025
+L +5V #PWR026
 U 1 1 591D5889
 P 8650 2250
-F 0 "#PWR025" H 8650 2100 50  0001 C CNN
+F 0 "#PWR026" H 8650 2100 50  0001 C CNN
 F 1 "+5V" H 8650 2390 50  0000 C CNN
 F 2 "" H 8650 2250 50  0000 C CNN
@@
 $EndComp
 $Comp
-L +3.3V #PWR026
+L +3.3V #PWR027
 U 1 1 591D5920
 P 8875 2250
-F 0 "#PWR026" H 8875 2100 50  0001 C CNN
+F 0 "#PWR027" H 8875 2100 50  0001 C CNN
 F 1 "+3.3V" H 8875 2390 50  0000 C CNN
 F 2 "" H 8875 2250 50  0000 C CNN
@@
 Wire Wire Line
 	6550 2700 6075 2700
+Text Label 6075 2700 0    60   ~ 0
+Mains_L
 Text Label 6075 2400 0    60   ~ 0
-Mains_L
-Text Label 6075 2700 0    60   ~ 0
 Mains_N
 Text HLabel 9150 2550 2    60   Output ~ 0

Commit message: PCB Update
Changed lines of the file:
@@
 Wire Wire Line
 	6550 2700 6075 2700
+Text Label 6075 2400 0    60   ~ 0
+Mains_L
 Text Label 6075 2700 0    60   ~ 0
-Mains_L
-Text Label 6075 2400 0    60   ~ 0
 Mains_N
 Text HLabel 9150 2550 2    60   Output ~ 0
