File: HW/PWRMET_24G.kicad_pcb (KiCad board)
At the start: 2 copper layers, 50 x 50 mm, 57 parts, among them P1 CONN_BOOT, P2 CONN_SWD, P3 IN, P4 OUT, P5 CONN_01X04, Q1 2N7002, SW1 SW_RST, U1 STM32F030F4Px, U2 nRF24L01_MODULE, U3 HLW8012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

Commit message: PCB Upd
Parts:
- moved C4 127.1 mm to (103.1, 77.2), turned to 270 degrees
- moved C5 115.7 mm to (95.2, 77.2), turned to 90 degrees
- moved C1 115.5 mm to (117.9, 77.0)
- moved R1 110.0 mm to (112.0, 77.2)
- moved U1 109.1 mm to (112.0, 85.3)
- moved P1 108.4 mm to (105.9, 77.2), turned to 90 degrees
- moved C2 108.2 mm to (119.6, 80.0)
- moved D1 105.8 mm to (87.6, 102.6)
- moved C3 103.1 mm to (97.3, 99.1), turned to 180 degrees
- moved R27 98.2 mm to (111.5, 114.0), turned to 180 degrees
- moved R3 96.3 mm to (91.7, 102.6), turned to 180 degrees
- moved R22 91.1 mm to (115.6, 114.0)
- moved C12 90.0 mm to (122.2, 113.8), turned to 90 degrees
- moved R2 89.9 mm to (104.4, 99.1)
- moved R28 89.8 mm to (110.8, 98.6)
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Connections:
- C11 pad 1: /RS485_ISOL/A -> /RS485_ISOL/PISO
- C12 pad 1: /RS485_ISOL/A -> /RS485_ISOL/PISO
- R20 pad 2: /RS485_ISOL/A -> /RS485_ISOL/PISO
- U4 pad 4: /RS485_ISOL/A -> /RS485_ISOL/PISO
- U5 pad 8: /RS485_ISOL/A -> /RS485_ISOL/PISO
- U6 pad 4: /RS485_ISOL/A -> /RS485_ISOL/PISO
- U7 pad 1: /RS485_ISOL/A -> /RS485_ISOL/PISO

Commit message: SCH&PCB Update
Parts:
- added D2: PLS_LED, LEDs:LED_D5.0mm, F.Cu at (121.5, 94.8)
- added R29: 1K, Resistors_SMD:R_0805, F.Cu at (115.8, 95.0)
- moved R19 94.2 mm to (101.5, 87.4), turned to 180 degrees
- moved R23 92.4 mm to (114.3, 120.4)
- moved R18 89.1 mm to (101.5, 89.4), turned to 180 degrees
- moved R17 88.9 mm to (101.5, 91.4), turned to 180 degrees
- moved R24 83.4 mm to (111.1, 120.4)
- moved R20 80.9 mm to (117.4, 120.4)
- moved R14 80.2 mm to (95.1, 88.5), turned to 90 degrees
- moved Q1 74.7 mm to (98.2, 92.2), turned to 180 degrees
- moved C1 10.7 mm to (107.7, 80.2), turned to 180 degrees
- moved C2 7.71 mm to (112.0, 79.2), turned to 180 degrees
- moved U1 4.39 mm to (107.6, 84.9), turned to 180 degrees
- moved R22 1.27 mm to (116.2, 112.9)
- moved R27 1.27 mm to (112.1, 112.9)
- moved U5 1.27 mm to (114.1, 116.7)
- moved C11 0.47 mm to (123.5, 113.7)
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Connections:
- PS1 pad 1: /HLW8012/Mains_L -> GND
- PS1 pad 2: GND -> /HLW8012/Mains_L
- U1 pad 3: (no net) -> /STM32_NRF24/PLS_OUT
Routing:
- net +3V3: track 0.00 -> 118.7 mm, vias 0 -> 7
- net GND: track 0.00 -> 91.5 mm, vias 0 -> 7
- net +5V: track 0.00 -> 49.7 mm, vias 0 -> 3
- net /HLW8012/Mains_L: track 0.00 -> 36.6 mm
- net /RS485_ISOL/PISO: track 0.00 -> 31.1 mm, vias 0 -> 2
- net /RS485_ISOL/GISO: track 0.00 -> 30.8 mm, vias 0 -> 5
- net /STM32_NRF24/NRST: track 0.00 -> 24.4 mm, vias 0 -> 2
- net /RS485_ISOL/DE: track 0.00 -> 22.8 mm, vias 0 -> 2
- net /STM32_NRF24/BOOT0: track 0.00 -> 22.4 mm, vias 0 -> 2
- net /RS485_ISOL/RX: track 0.00 -> 20.8 mm
- net /RS485_ISOL/TX: track 0.00 -> 19.2 mm, vias 0 -> 2
- net /RS485_ISOL/12V_ISO: track 0.00 -> 18.8 mm
- net /STM32_NRF24/SYS_SWDIO: track 0.00 -> 17.3 mm
- net /HLW8012/V2P: track 0.00 -> 16.2 mm
- net /STM32_NRF24/SYS_SWCLK: track 0.00 -> 16.1 mm
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- added copper zone on B.Cu, net /RS485_ISOL/GISO
- added copper zone on B.Cu, net GND
Other:
- rule trace_min: 0.2 -> 0.25

Commit message: PCB Gerbers
Parts:
- added REF**: KiCAD Logo, Symbols:Symbol_KiCAD-Logo_CopperAndSilkScreenTop, B.Cu at (85.8, 109.4)
- added REF***: OSHW-Logo2_9.8x8mm_SilkScreen, Symbols:OSHW-Logo2_9.8x8mm_SilkScreen, B.Cu at (97.1, 109.9)
Other:
- board text added: "!HIGH VOLTAGE! NON ISOLATED"
- board text added: "10count/KWh"
- board text added: "16A"
- board text added: "5V 700mA SMPSU"
- board text added: "BOOT0"
- board text added: "Energy Meter RF/485 V1.0 BK 2017"
- board text added: "INPUT"
- board text added: "NRF24L01"
- board text added: "OUTPUT"
- board text added: "R6 10A or R7 16A Max"
- board text added: "R6 or R7 .001R"
- board text added: "RS485 Conn: 1 - 12V 2 - 485 B 3 - 485 A 4 - GND"
- board text added: "SWD Conn: 1 - 3.3V 2 - SWDIO 3 - SWDCLK 4 - GND"
- board text added: "https://github.com/bklemencz/PWRMET_24G"

Commit message: PCB Update
Parts:
- moved C6 4.42 mm to (91.7, 94.6)
- moved Q1 3.32 mm to (94.8, 92.4)
- moved R17 2.27 mm to (99.8, 92.9)
- moved C7 1.52 mm to (91.7, 96.8)
- moved R11 1.47 mm to (91.7, 99.0)
Connections:
- PS1 pad 1: GND -> /HLW8012/Mains_L
- PS1 pad 2: /HLW8012/Mains_L -> GND
Routing:
- net /HLW8012/Mains_L: track 36.6 -> 46.6 mm
- net /HLW8012/V1P: track 9.20 -> 14.4 mm
- net GND: track 91.5 -> 94.4 mm
- net /HLW8012/V1N: track 15.6 -> 17.9 mm
Other:
- net class Mains added: clearance 0.8, trace_width 0.25, via_dia 0.6, via_drill 0.4
- rule pad_to_mask_clearance: 0.2 -> 0
- board text added: "100count/KWh"
- board text removed: "10count/KWh"
